File: Dimmer.sch (KiCad schematic (older format))
At the start: 21 parts, among them IC1 TTP224B-BSBN, J1 Reset, J2 Prog, J3 Conn_01x04, J4 Mode, J5 Load_cntrl, J6 Detect_null, U1 ESP-07, k1 Key, k2 Key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

Commit message: Add files via upload
Parts:
- k1: footprint Touch_pad:Touch_pad -> Touch_pad:TestPoint_Pad_2.5x2.5sm
- k2, k3: footprint Touch_pad:Touch_pad -> Touch_pad:TestPoint_Pad_1.0x1.0sm
Changed lines of the file:
@@
 F 0 "k1" H 3908 3775 50  0000 C CNN
 F 1 "Key" H 3908 3684 50  0000 C CNN
-F 2 "Touch_pad:Touch_pad" H 3950 3650 50  0001 C CNN
+F 2 "Touch_pad:TestPoint_Pad_2.5x2.5sm" H 3950 3650 50  0001 C CNN
 F 3 "" H 3950 3650 50  0001 C CNN
 	1    3950 3650
@@
 F 0 "k2" H 4308 3775 50  0000 C CNN
 F 1 "Key" H 4308 3684 50  0000 C CNN
-F 2 "Touch_pad:Touch_pad" H 4350 3650 50  0001 C CNN
+F 2 "Touch_pad:TestPoint_Pad_1.0x1.0sm" H 4350 3650 50  0001 C CNN
 F 3 "" H 4350 3650 50  0001 C CNN
 	1    4350 3650
@@
 F 0 "k3" H 4658 3775 50  0000 C CNN
 F 1 "Key" H 4658 3684 50  0000 C CNN
-F 2 "Touch_pad:Touch_pad" H 4700 3650 50  0001 C CNN
+F 2 "Touch_pad:TestPoint_Pad_1.0x1.0sm" H 4700 3650 50  0001 C CNN
 F 3 "" H 4700 3650 50  0001 C CNN
 	1    4700 3650

Commit message: Add files via upload
Parts:
- removed C3: 30p, Capacitor_SMD:C_0603_1608Metric, symbol pspice:C
- removed C5: 100mk, Capacitor_SMD:C_1210_3225Metric, symbol pspice:C
- removed IC1: TTP224B-BSBN, TTP224B-BSBN:SOP64P600X175-16N, symbol TTP224B-BSBN:TTP224B-BSBN
- removed J1: Reset, Connector_PinHeader_2.54mm:PinHeader_1x02_P2.54mm_Vertical, symbol Connector_Generic:Conn_01x02
- removed U1: ESP-07, RF_Module:ESP-07, symbol RF_Module:ESP-07
- added C11: 0.33mk, Capacitor_SMD:C_1210_3225Metric, symbol pspice:C
- added C8: 0.1mk, Capacitor_SMD:C_1210_3225Metric, symbol pspice:C
- added D1, D2: BAV99, Package_TO_SOT_SMD:SOT-23, symbol Diode:BAV99
- added D3: BZX84Cxx, Diode_SMD:D_SOT-23_ANK, symbol Diode:BZX84Cxx
- added D4: 1N4148WT, Diode_SMD:D_SOD-523, symbol Diode:1N4148WT
- added D5: BLUE, LED_SMD:LED_0603_1608Metric, symbol Device:LED
- added D6: RED, LED_SMD:LED_0603_1608Metric, symbol Device:LED
- added J1: 220to12, Converter_ACDC:Converter_ACDC_MeanWell_IRM-02-xx_THT, symbol w_connectors:HEADER_2x2
- added J10: Detect_nullA, Connector:FanPinHeader_1x03_P2.54mm_Vertical, symbol Connector_Generic:Conn_01x03
- added J11: 220v_OUT, Connector_Phoenix_MC_HighVoltage:PhoenixContact_MC_1,5_2-G-5.08_1x02_P5.08mm_Horizontal, symbol Connector_Generic:Conn_01x02
- added J12: Load_cntrlA, Connector:FanPinHeader_1x03_P2.54mm_Vertical, symbol Connector_Generic:Conn_01x03
- added J13, J8: ADC, Touch_pad:polz_razjem, symbol Connector_Generic:Conn_01x01
- added J14, J15, J16, J17, J18, J19: Conn_01x01, Touch_pad:polz_razjem, symbol Connector_Generic:Conn_01x01
- added J22: SPI, Connector_PinHeader_2.54mm:PinHeader_1x04_P2.54mm_Vertical_SMD_Pin1Right, symbol Connector_Generic:Conn_01x04
- added J7: I2C, Connector_PinHeader_2.54mm:PinHeader_1x04_P2.54mm_Horizontal, symbol Connector_Generic:Conn_01x03
- added J9: 220v_IN, Connector_Phoenix_MC_HighVoltage:PhoenixContact_MC_1,5_2-G-5.08_1x02_P5.08mm_Horizontal, symbol Connector_Generic:Conn_01x02
- added Q1, Q2: IRFP460APBF, Package_TO_SOT_THT:TO-220-3_Horizontal_TabDown, symbol Transistor_FET:IRF4905
- added Q3: BC807, Package_TO_SOT_SMD:SOT-23, symbol Transistor_BJT:BC807
- added R10: 220, Resistor_SMD:R_0603_1608Metric, symbol Device:R
- added R11, R12: 220, Resistor_SMD:R_1206_3216Metric, symbol Device:R
- added R13, R9: 10k, Resistor_SMD:R_0603_1608Metric, symbol Device:R
- added R6: 120k 0.25W, Resistor_SMD:R_0603_1608Metric, symbol Device:R
- added R7: 220 1W, Resistor_SMD:R_0603_1608Metric, symbol Device:R
- added R8: 330k 0.25W, Resistor_SMD:R_0603_1608Metric, symbol Device:R
- added SW1, SW2: SW_Push, Button_Switch_SMD:SW_DIP_SPSTx01_Slide_6.7x4.1mm_W6.73mm_P2.54mm_LowProfile_JPin, symbol Switch:SW_Push
- added TH1, TH2: Thermistor_NTC, Resistor_SMD:R_1206_3216Metric_Pad1.30x1.75mm_HandSolder, symbol Device:Thermistor_NTC
- added U1: FAN3268, Package_SO:SOIC-8_3.9x4.9mm_P1.27mm, symbol Driver_FET:FAN3268
- added U2: ESP32-WROOM-32D, RF_Module:ESP32-WROOM-32, symbol RF_Module:ESP32-WROOM-32D
- added U3: L78L33_SO8, Package_SO:SOIC-8_3.9x4.9mm_P1.27mm, symbol Regulator_Linear:L78L33_SO8
- added U4: TLP185, Package_SO:SOIC-4_4.55x3.7mm_P2.54mm, symbol Isolator:TLP185
- added k4, k5, k6, k7: Key, Touch_pad:TestPoint_Pad_1.0x1.0sm, symbol Touchpad:Key
- C1: value 30p -> 0.01mk; footprint Capacitor_SMD:C_0603_1608Metric -> Capacitor_SMD:C_1210_3225Metric
- C2: value 30p -> 0.47mk; footprint Capacitor_SMD:C_0603_1608Metric -> Capacitor_SMD:C_1210_3225Metric
- J2: footprint Connector_PinHeader_2.54mm:PinHeader_1x02_P2.54mm_Vertical -> Connector_PinHeader_2.54mm:PinHeader_1x02_P2.54mm_Vertical_SMD_Pin1Left
- J3: value Conn_01x04 -> UART0; footprint Connector_PinHeader_2.54mm:PinHeader_1x04_P2.54mm_Vertical -> Connector_PinHeader_2.54mm:PinHeader_1x04_P2.54mm_Horizontal
- J4: footprint Connector_PinHeader_2.54mm:PinHeader_1x02_P2.54mm_Vertical -> Connector_PinHeader_2.54mm:PinHeader_1x04_P2.54mm_Vertical_SMD_Pin1Left
- J5, J6: footprint Connector_PinHeader_2.54mm:PinHeader_1x03_P2.54mm_Vertical -> Connector:FanPinHeader_1x03_P2.54mm_Vertical
- R4: value 10k -> 120k 0.25W
Connections:
- net labels added: +12V, BLUE, GPIO17, GPIO26, GPIO32, GPIO35, MOSI, Mode, RED, cntrl
- net labels removed: GPIO15, GPIO4
- wire segments 80 -> 133
- no-connect marks 10 -> 4
Other:
- moved on the sheet: C4, J2, J3, J4, J5, J6, R1, R2, R3, R5

Commit message: Add files via upload
Parts:
- removed Q1, Q2: IRFP460APBF, Package_TO_SOT_THT:TO-220-3_Horizontal_TabDown, symbol Transistor_FET:IRF4905
- removed U1: FAN3268, Package_SO:SOIC-8_3.9x4.9mm_P1.27mm, symbol Driver_FET:FAN3268
- added D7: Fan3100tsx, Package_TO_SOT_SMD:SOT-23-5, symbol Dimmer-rescue:Fan3100tsx-Fan3100TSX
- added Q1, Q2: IRFP460APBF, Package_TO_SOT_THT:TO-247-3_Horizontal_TabDown, symbol Transistor_FET:C3M0280090D
- D5, D6: footprint LED_SMD:LED_0603_1608Metric -> LED_THT:LED_D3.0mm_Clear
- J1: symbol w_connectors:HEADER_2x2 -> Dimmer-rescue:HEADER_2x2-w_connectors
- k1, k2, k3, k4, k5, k6, k7: symbol Touchpad:Key -> Dimmer-rescue:Key-Touchpad
Connections:
- no-connect marks 4 -> 0
Changed lines of the file:
@@
 $EndComp
 $Comp
-L Touchpad:Key k3
+L Dimmer-rescue:Key-Touchpad k3
 U 1 1 60C69E9B
 P 8500 5250
@@
 $EndComp
 $Comp
-L Touchpad:Key k2
+L Dimmer-rescue:Key-Touchpad k2
 U 1 1 60C693B3
 P 8500 3450
@@
 $EndComp
 $Comp
-L Touchpad:Key k1
+L Dimmer-rescue:Key-Touchpad k1
 U 1 1 60C6833A
 P 8500 3650
@@
 $EndComp
 $Comp
-L Touchpad:Key k5
+L Dimmer-rescue:Key-Touchpad k5
 U 1 1 60DCD999
 P 8500 3950
@@
 $EndComp
 $Comp
-L Touchpad:Key k4
+L Dimmer-rescue:Key-Touchpad k4
 U 1 1 60DCDD4E
 P 8500 3850
@@
 $EndComp
 $Comp
-L Touchpad:Key k6
+L Dimmer-rescue:Key-Touchpad k6
 U 1 1 60DCE2FD
 P 8500 4050
@@
 $EndComp
 $Comp
-L Touchpad:Key k7
+L Dimmer-rescue:Key-Touchpad k7
 U 1 1 60DCEBF7
 P 8500 5150
@@
 Wire Wire Line
 	6100 1550 6150 1550
-NoConn ~ 4050 3100
-NoConn ~ 4050 3200
-$Comp
-L Driver_FET:FAN3268 U1
-U 1 1 60EFDBA9
-P 3650 3000
-F 0 "U1" H 3650 3681 50  0000 C CNN
-F 1 "FAN3268" H 3650 3590 50  0000 C CNN
-F 2 "Package_SO:SOIC-8_3.9x4.9mm_P1.27mm" H 3700 2550 50  0001 L CNN
-F 3 "http://www.onsemi.com/pub/Collateral/FAN3268T_F085-D.PDF" H 3650 3100 50  0001 C CNN
-	1    3650 3000
-	-1   0    0    -1
-$EndComp
-NoConn ~ 4050 2900
-NoConn ~ 3250 2900
 $Comp
 L Device:R R4
@@
 $EndComp
 $Comp
-L Transistor_FET:IRF4905 Q2
-U 1 1 60F2E091
-P 2800 3050
-F 0 "Q2" H 3005 3004 50  0000 L CNN
-F 1 "IRFP460APBF" H 3005 3095 50  0000 L CNN
-F 2 "Package_TO_SOT_THT:TO-220-3_Horizontal_TabDown" H 3000 2975 50  0001 L CIN
-F 3 "http://www.infineon.com/dgdl/irf4905.pdf?fileId=5546d462533600a4015355e32165197c" H 2800 3050 50  0001 L CNN
-	1    2800 3050
-	-1   0    0    1
-$EndComp
-$Comp
-L Transistor_FET:IRF4905 Q1
-U 1 1 60F3259D
-P 2800 2500
-F 0 "Q1" H 3005 2546 50  0000 L CNN
-F 1 "IRFP460APBF" H 3005 2455 50  0000 L CNN
-F 2 "Package_TO_SOT_THT:TO-220-3_Horizontal_TabDown" H 3000 2425 50  0001 L CIN
-F 3 "http://www.infineon.com/dgdl/irf4905.pdf?fileId=5546d462533600a4015355e32165197c" H 2800 2500 50  0001 L CNN
-	1    2800 2500
-	-1   0    0    -1
-$EndComp
-$Comp
 L pspice:C C1
 U 1 1 60F3CB59
@@
 	3000 2500 3000 2800
 $Comp
-L w_connectors:HEADER_2x2 J1
+L Dimmer-rescue:HEADER_2x2-w_connectors J1
 U 1 1 60F5D81B
 P 1600 3750
@@
 L power:GND #PWR0107
 U 1 1 60F5EA64
-P 3650 3500
-F 0 "#PWR0107" H 3650 3250 50  0001 C CNN
-F 1 "GND" H 3655 3327 50  0000 C CNN
-F 2 "" H 3650 3500 50  0001 C CNN
-F 3 "" H 3650 3500 50  0001 C CNN
-	1    3650 3500
+P 3250 3000
+F 0 "#PWR0107" H 3250 2750 50  0001 C CNN
+F 1 "GND" H 3255 2827 50  0000 C CNN
+F 2 "" H 3250 3000 50  0001 C CNN
+F 3 "" H 3250 3000 50  0001 C CNN
+	1    3250 3000
 	1    0    0    -1
 $EndComp
@@
 Wire Wire Line
 	6350 1350 6100 1350
-Text GLabel 4050 2800 2    50   Input ~ 0
+Text GLabel 4000 2950 2    50   Input ~ 0
 cntrl
 $Comp
 L power:+12V #PWR0118
 U 1 1 61074A57
-P 3650 2500
-F 0 "#PWR0118" H 3650 2350 50  0001 C CNN
-F 1 "+12V" H 3665 2673 50  0000 C CNN
-F 2 "" H 3650 2500 50  0001 C CNN
-F 3 "" H 3650 2500 50  0001 C CNN
-	1    3650 2500
+P 4000 2800
+F 0 "#PWR0118" H 4000 2650 50  0001 C CNN
+F 1 "+12V" H 4015 2973 50  0000 C CNN
+F 2 "" H 4000 2800 50  0001 C CNN
+F 3 "" H 4000 2800 50  0001 C CNN
+	1    4000 2800
 	1    0    0    -1
 $EndComp
@@
 F 0 "D5" V 10239 5682 50  0000 R CNN
 F 1 "BLUE" V 10148 5682 50  0000 R CNN
-F 2 "LED_SMD:LED_0603_1608Metric" H 10200 5800 50  0001 C CNN
+F 2 "LED_THT:LED_D3.0mm_Clear" H 10200 5800 50  0001 C CNN
 F 3 "~" H 10200 5800 50  0001 C CNN
 	1    10200 5800
@@
 F 0 "D6" V 10639 5682 50  0000 R CNN
 F 1 "RED" V 10548 5682 50  0000 R CNN
-F 2 "LED_SMD:LED_0603_1608Metric" H 10600 5800 50  0001 C CNN
+F 2 "LED_THT:LED_D3.0mm_Clear" H 10600 5800 50  0001 C CNN
 F 3 "~" H 10600 5800 50  0001 C CNN
 	1    10600 5800
@@
 Text GLabel 8450 5650 2    50   Input ~ 0
 GPIO35
+$Comp
+L Transistor_FET:C3M0280090D Q2
+U 1 1 60DBB938
+P 2800 3050
+F 0 "Q2" H 3005 3004 50  0000 L CNN
+F 1 "IRFP460APBF" H 3005 3095 50  0000 L CNN
+F 2 "Package_TO_SOT_THT:TO-247-3_Horizontal_TabDown" H 2800 3050 50  0001 C CIN
+F 3 "https://www.wolfspeed.com/media/downloads/825/C3M0280090D.pdf" H 2800 3050 50  0001 L CNN
+	1    2800 3050
+	-1   0    0    1
+$EndComp
+$Comp
+L Transistor_FET:C3M0280090D Q1
+U 1 1 60DDB34A
+P 2800 2500
+F 0 "Q1" H 3005 2546 50  0000 L CNN
+F 1 "IRFP460APBF" H 3005 2455 50  0000 L CNN
+F 2 "Package_TO_SOT_THT:TO-247-3_Horizontal_TabDown" H 2800 2500 50  0001 C CIN
+F 3 "https://www.wolfspeed.com/media/downloads/825/C3M0280090D.pdf" H 2800 2500 50  0001 L CNN
+	1    2800 2500
+	-1   0    0    -1
+$EndComp
+$Comp
+L Dimmer-rescue:Fan3100tsx-Fan3100TSX D7
+U 1 1 60DE385E
+P 3600 2700
+F 0 "D7" H 3625 2825 50  0000 C CNN
+F 1 "Fan3100tsx" H 3625 2734 50  0000 C CNN
+F 2 "Package_TO_SOT_SMD:SOT-23-5" H 3600 2700 50  0001 C CNN
+F 3 "" H 3600 2700 50  0001 C CNN
+	1    3600 2700
+	1    0    0    -1
+$EndComp
+$Comp
+L power:GND #PWR0124
+U 1 1 60DEA9D0
+P 4000 3050
+F 0 "#PWR0124" H 4000 2800 50  0001 C CNN
+F 1 "GND" H 4005 2877 50  0000 C CNN
+F 2 "" H 4000 3050 50  0001 C CNN
+F 3 "" H 4000 3050 50  0001 C CNN
+	1    4000 3050
+	1    0    0    -1
+$EndComp
 $EndSCHEMATC
