File: Dimmer.sch (KiCad schematic (older format))
At the start: 58 parts, among them J1 220to12, J11 220v_OUT, J16 Conn_01x06, J2 Prog, J22 SPI, J3 UART0, J4 Conn_01x06, J9 220v_IN, Q1 IRFP460APBF, Q2 IRFP460APBF, Q3 BC807, U1 LM75B, U2 ESP32-WROOM-32D, U22 AMS1117-3.3, U4 TLP185, k2 Key, k3 Key, k4 Key, k5 Key, k6 Key, k7 Key

Commit message: Замена С1, блок 220-12 поставлен вертикально
Parts:
- C1: footprint Capacitor_SMD:C_0805_2012Metric -> Capacitor_THT:C_Rect_L10.0mm_W2.5mm_P7.50mm_MKS4
Connections:
- wire segments 130 -> 138
Other:
- moved on the sheet: J1
Changed lines of the file:
@@
 L Dimmer-rescue:HEADER_2x2-w_connectors-Dimmer-rescue-Dimmer-rescue J1
 U 1 1 60F5D81B
-P 1600 3750
-F 0 "J1" H 1600 4037 60  0000 C CNN
-F 1 "220to12" H 1600 3931 60  0000 C CNN
-F 2 "SMout:oblast_bp" H 1600 3750 60  0001 C CNN
-F 3 "" H 1600 3750 60  0000 C CNN
-	1    1600 3750
-	1    0    0    -1
-$EndComp
-Wire Wire Line
-	1450 3700 1000 3700
+P 1780 3760
+F 0 "J1" H 1780 4047 60  0000 C CNN
+F 1 "220to12" H 1780 3941 60  0000 C CNN
+F 2 "SMout:oblast_bp" H 1780 3760 60  0001 C CNN
+F 3 "" H 1780 3760 60  0000 C CNN
+	1    1780 3760
+	1    0    0    -1
+$EndComp
 Wire Wire Line
 	1000 3700 1000 2300
@@
 Wire Wire Line
 	900  2100 900  3150
-Wire Wire Line
-	900  3800 1450 3800
 Wire Wire Line
 	800  3150 900  3150
 Connection ~ 900  3150
 Wire Wire Line
-	900  3150 900  3800
+	900  3150 900  3795
 Connection ~ 1000 2300
 $Comp
 L power:GND #PWR0117
 U 1 1 60FBD5CD
-P 1750 3800
-F 0 "#PWR0117" H 1750 3550 50  0001 C CNN
-F 1 "GND" H 1755 3627 50  0000 C CNN
-F 2 "" H 1750 3800 50  0001 C CNN
-F 3 "" H 1750 3800 50  0001 C CNN
-	1    1750 3800
+P 1930 3810
+F 0 "#PWR0117" H 1930 3560 50  0001 C CNN
+F 1 "GND" H 1935 3637 50  0000 C CNN
+F 2 "" H 1930 3810 50  0001 C CNN
+F 3 "" H 1930 3810 50  0001 C CNN
+	1    1930 3810
 	1    0    0    -1
 $EndComp
@@
 L power:+12V #PWR0123
 U 1 1 61075161
-P 1750 3700
-F 0 "#PWR0123" H 1750 3550 50  0001 C CNN
-F 1 "+12V" H 1765 3873 50  0000 C CNN
-F 2 "" H 1750 3700 50  0001 C CNN
-F 3 "" H 1750 3700 50  0001 C CNN
-	1    1750 3700
+P 1930 3710
+F 0 "#PWR0123" H 1930 3560 50  0001 C CNN
+F 1 "+12V" H 1945 3883 50  0000 C CNN
+F 2 "" H 1930 3710 50  0001 C CNN
+F 3 "" H 1930 3710 50  0001 C CNN
+	1    1930 3710
 	1    0    0    -1
 $EndComp
@@
 F 0 "C1" H 1125 3090 50  0000 L CNN
 F 1 "0.1 mk" H 1040 2910 50  0000 L CNN
-F 2 "Capacitor_SMD:C_0805_2012Metric" H 1315 3000 50  0001 C CNN
+F 2 "Capacitor_THT:C_Rect_L10.0mm_W2.5mm_P7.50mm_MKS4" H 1315 3000 50  0001 C CNN
 F 3 "~" H 1315 3000 50  0001 C CNN
 	1    1315 3000
@@
 Wire Wire Line
 	1315 3250 1880 3250
+Wire Wire Line
+	1630 3710 1545 3710
+Wire Wire Line
+	995  3700 1000 3700
+Wire Wire Line
+	1545 3700 1545 3710
+Connection ~ 1000 3700
+Wire Wire Line
+	1000 3700 1545 3700
+Connection ~ 1545 3710
+Wire Wire Line
+	1545 3710 1540 3710
+Wire Wire Line
+	900  3795 1630 3795
+Wire Wire Line
+	1630 3795 1630 3805
+Wire Wire Line
+	1630 3805 1635 3805
+Connection ~ 900  3795
+Wire Wire Line
+	900  3795 900  3800
+Wire Wire Line
+	1630 3810 1630 3805
+Connection ~ 1630 3805
 $EndSCHEMATC
