File: Dimmer.kicad_pcb (KiCad board)
At the start: 2 copper layers, 63.9 x 63.9 mm, 21 parts, among them IC1 TTP224B-BSBN, J1 Reset, J2 Prog, J3 Conn_01x04, J4 Mode, J5 Load_cntrl, J6 Detect_null, U1 ESP-07, k1 Key, k2 Key, k3 Key

Commit message: Add files via upload
Parts:
- removed C3: 30p, Capacitor_SMD:C_0603_1608Metric
- removed C5: 100mk, Capacitor_SMD:C_1210_3225Metric
- removed IC1: TTP224B-BSBN, TTP224B-BSBN:SOP64P600X175-16N
- added C11: 0.33mk, Capacitor_SMD:C_1210_3225Metric, F.Cu at (232.0, 100.5)
- added C8: 0.1mk, Capacitor_SMD:C_1210_3225Metric, F.Cu at (228.0, 92.0)
- added D1: BAV99, Package_TO_SOT_SMD:SOT-23, F.Cu at (233.0, 125.7)
- added D2: BAV99, Package_TO_SOT_SMD:SOT-23, F.Cu at (228.7, 130.3)
- added D3: BZX84Cxx, Diode_SMD:D_SOT-23_ANK, B.Cu at (223.0, 121.0)
- added D4: 1N4148WT, Diode_SMD:D_SOD-523, F.Cu at (233.0, 117.3)
- added D5: BLUE, LED_SMD:LED_0603_1608Metric, B.Cu at (105.5, 127.4)
- added D6: RED, LED_SMD:LED_0603_1608Metric, B.Cu at (168.5, 127.6)
- added J10: Detect_nullA, Connector:FanPinHeader_1x03_P2.54mm_Vertical, B.Cu at (230.8, 108.3)
- added J11: 220v_OUT, Touch_pad:220V_1x02_P5.08mm_Horizontal, F.Cu at (215.7, 125.9)
- added J12: Load_cntrlA, Connector:FanPinHeader_1x03_P2.54mm_Vertical, B.Cu at (192.7, 113.5)
- added J13: ADC, Touch_pad:polz_razjem, F.Cu at (109.0, 85.0)
- added J14: Conn_01x01, Touch_pad:polz_razjem, F.Cu at (157.0, 140.0)
- added J15: Conn_01x01, Touch_pad:polz_razjem, F.Cu at (160.0, 138.0)
- added J16: Conn_01x01, Touch_pad:polz_razjem, F.Cu at (115.0, 138.0)
- added J17: Conn_01x01, Touch_pad:polz_razjem, F.Cu at (118.0, 140.0)
- added J18: Conn_01x01, Touch_pad:polz_razjem, F.Cu at (154.0, 138.0)
- added J19: Conn_01x01, Touch_pad:polz_razjem, F.Cu at (121.0, 138.0)
- added J22: SPI, Connector_PinHeader_2.54mm:PinHeader_1x04_P2.54mm_Vertical_SMD_Pin1Right, F.Cu at (155.7, 96.3)
- added J7: I2C, Connector_PinHeader_2.54mm:PinHeader_1x03_P2.54mm_Horizontal, F.Cu at (167.0, 81.9)
- added J8: ADC, Touch_pad:polz_razjem, F.Cu at (111.0, 83.0)
- added J9: 220v_IN, Touch_pad:220V_1x02_P5.08mm_Horizontal, F.Cu at (203.7, 125.9)
- added Q1: IRFP460APBF, Package_TO_SOT_THT:TO-220-3_Horizontal_TabDown, B.Cu at (213.0, 119.0)
- added Q2: IRFP460APBF, Package_TO_SOT_THT:TO-220-3_Horizontal_TabDown, F.Cu at (218.5, 116.7)
- added Q3: BC807, Package_TO_SOT_SMD:SOT-23, B.Cu at (227.1, 118.0)
- added R10: 220, Resistor_SMD:R_0603_1608Metric, B.Cu at (231.0, 117.2)
- added R11: 220, Resistor_SMD:R_1206_3216Metric, F.Cu at (113.0, 98.5)
- added R12: 220, Resistor_SMD:R_1206_3216Metric, F.Cu at (147.0, 111.5)
- added R13: 10k, Resistor_SMD:R_0603_1608Metric, F.Cu at (131.0, 123.2)
- added R6: 120k 0.25W, Resistor_SMD:R_0603_1608Metric, F.Cu at (226.0, 124.8)
- added R7: 220 1W, Resistor_SMD:R_0603_1608Metric, B.Cu at (217.0, 109.2)
- added R8: 330k 0.25W, Resistor_SMD:R_1206_3216Metric, F.Cu at (230.0, 122.0)
- added R9: 10k, Resistor_SMD:R_0603_1608Metric, F.Cu at (223.0, 91.8)
- added SW1: SW_Push, Button_Switch_SMD:SW_DIP_SPSTx01_Slide_6.7x4.1mm_W6.73mm_P2.54mm_LowProfile_JPin, B.Cu at (107.0, 135.0)
- added SW2: SW_Push, Button_Switch_SMD:SW_DIP_SPSTx01_Slide_6.7x4.1mm_W6.73mm_P2.54mm_LowProfile_JPin, B.Cu at (167.0, 135.0)
- added TH1: Thermistor_NTC, Resistor_SMD:R_1206_3216Metric_Pad1.30x1.75mm_HandSolder, F.Cu at (219.0, 91.0)
- added TH2: Thermistor_NTC, Resistor_SMD:R_1206_3216Metric_Pad1.30x1.75mm_HandSolder, F.Cu at (131.0, 117.5)
- added U2: ESP32-WROOM-32D, RF_Module:ESP32-WROOM-32, F.Cu at (138.0, 95.0)
- added U3: L78L33_SO8, Package_SO:SOIC-8_3.9x4.9mm_P1.27mm, B.Cu at (221.5, 101.6)
- added U4: TLP185, Package_SO:SOIC-4_4.55x3.7mm_P2.54mm, B.Cu at (225.0, 110.0)
- added k4: Key, Touch_pad:TestPoint_Pad_1.0x1.0sm, B.Cu at (107.0, 128.0)
- added k5: Key, Touch_pad:TestPoint_Pad_1.0x1.0sm, B.Cu at (137.0, 144.0)
- added k6: Key, Touch_pad:TestPoint_Pad_1.0x1.0sm, B.Cu at (122.0, 101.0)
- added k7: Key, Touch_pad:TestPoint_Pad_1.0x1.0sm, B.Cu at (138.0, 92.0)
- C1: value 30p -> 0.01mk; footprint Capacitor_SMD:C_0603_1608Metric -> Capacitor_SMD:C_1210_3225Metric; moved to B.Cu
- C2: value 30p -> 0.47mk; footprint Capacitor_SMD:C_0603_1608Metric -> Capacitor_SMD:C_1210_3225Metric
- J1: value Reset -> 220to12; footprint Connector_PinHeader_2.54mm:PinHeader_1x02_P2.54mm_Vertical -> Touch_pad:oblast_bp
- J2, J4: footprint Connector_PinHeader_2.54mm:PinHeader_1x02_P2.54mm_Vertical -> Connector_PinHeader_2.54mm:PinHeader_1x02_P2.54mm_Vertical_SMD_Pin1Left
- J3: value Conn_01x04 -> UART0; footprint Connector_PinHeader_2.54mm:PinHeader_1x04_P2.54mm_Vertical -> Connector_PinHeader_2.54mm:PinHeader_1x04_P2.54mm_Horizontal
- J5, J6: footprint Connector_PinHeader_2.54mm:PinHeader_1x03_P2.54mm_Vertical -> Connector:FanPinHeader_1x03_P2.54mm_Vertical
- R4: value 10k -> 120k 0.25W; moved to B.Cu
- U1: value ESP-07 -> FAN3268; footprint RF_Module:ESP-07 -> Package_SO:SOIC-8_3.9x4.9mm_P1.27mm; moved to B.Cu
- k1: footprint Touch_pad:TestPoint_Pad_2.5x2.5sm -> Touch_pad:TestPoint_Pad_1.0x1.0sm
- moved R4 95.2 mm to (234.5, 121.2), turned to 90 degrees
- moved J1 73.4 mm to (206.5, 105.0)
- moved U1 70.8 mm to (230.0, 100.0), turned to 270 degrees
- moved C2 61.2 mm to (228.0, 117.0), turned to 180 degrees
- moved R2 61.0 mm to (118.0, 86.8)
- moved C1 55.5 mm to (220.0, 108.5), turned to 270 degrees
- moved k3 46.4 mm to (137.0, 118.0), turned to 0 degrees
- moved C4 44.3 mm to (120.0, 81.5), turned to 90 degrees
- moved J4 41.8 mm to (148.3, 128.3), turned to 270 degrees
- moved R3 41.4 mm to (106.0, 80.0), turned to 45 degrees
- moved R1 38.9 mm to (115.0, 81.5), turned to 90 degrees
- moved J3 36.0 mm to (156.4, 78.0), turned to 90 degrees
- moved J2 27.0 mm to (155.3, 116.7)
- moved J6 25.0 mm to (156.0, 105.5)
- moved R5 20.6 mm to (157.2, 84.0)
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Connections:
- C1 pad 2: GND -> Net-(C1-Pad2)
- C2 pad 2: GND -> Net-(C2-Pad2)
- J1 pad 2: GND -> +12V
- J3 pad 1: Net-(J3-Pad1) -> +3V3
- J3 pad 3: GND -> Net-(J3-Pad3)
- J3 pad 4: +3V3 -> GND
- J4 pad 1: Net-(J4-Pad1) -> Mode
- J4 pad 2: GND -> Net-(J4-Pad2)
- J5 pad 2: +3V3 -> GPIO26
- J5 pad 3: GPIO15 -> GPIO32
- J6 pad 1: GPIO4 -> GPIO17
- R1 pad 2: Net-(R1-Pad2) -> GPIO35
- R2 pad 2: Net-(J2-Pad1) -> Net-(R2-Pad2)
- R3 pad 1: Net-(R1-Pad2) -> GPIO35
- R4 pad 1: +3V3 -> Net-(D1-Pad3)
- R4 pad 2: Net-(R4-Pad2) -> Net-(J1-Pad1)
- R5 pad 2: Net-(J1-Pad1) -> Net-(J2-Pad1)
- U1 pad 1: Net-(J1-Pad1) -> Net-(U1-Pad1)
- U1 pad 2: Net-(R1-Pad2) -> cntrl
- U1 pad 3: Net-(R4-Pad2) -> GND
- U1 pad 6: Net-(IC1-Pad15) -> +12V
- U1 pad 8: +3V3 -> Net-(U1-Pad8)
- k1 pad 1: Net-(C1-Pad1) -> Net-(U2-Pad26)
- k2 pad 1: Net-(C2-Pad1) -> Net-(U2-Pad24)
Routing:
- net GND: track 159.2 -> 437.4 mm, vias 1 -> 4
- net +3V3: track 115.3 -> 248.5 mm, vias 8 -> 5
- net Net-(U2-Pad12): track 0.00 -> 99.9 mm, vias 0 -> 3
- net Net-(J2-Pad1): track 15.7 -> 115.1 mm, vias 0 -> 2
- net Net-(R2-Pad2): track 0.00 -> 88.7 mm, vias 0 -> 5
- net GPIO15: track 68.7 -> 0.00 mm
- net cntrl: track 0.00 -> 59.7 mm
- net Net-(J16-Pad1): track 0.00 -> 56.3 mm
- net Net-(J17-Pad1): track 0.00 -> 56.1 mm
- net +12V: track 0.00 -> 56.1 mm, vias 0 -> 1
- net Net-(J1-Pad3): track 0.00 -> 54.2 mm
- net Net-(J19-Pad1): track 0.00 -> 51.6 mm
- net Net-(U2-Pad13): track 0.00 -> 51.5 mm, vias 0 -> 1
- net MOSI: track 0.00 -> 51.4 mm, vias 0 -> 2
- net Net-(J1-Pad1): track 21.4 -> 72.8 mm, vias 0 -> 1
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- added copper zone on F.Cu, net GND
Other:
- board size 63.9 x 63.9 mm -> 132.8 x 68 mm
- net class Default: trace_width 0.6 -> 0.25
- rule trace_min: 0.3 -> 0.2
- rule via_min_drill: 0.2 -> 0.3
- rule via_min_size: 0.3 -> 0.4

Commit message: Add files via upload
Parts:
- removed U1: FAN3268, Package_SO:SOIC-8_3.9x4.9mm_P1.27mm
- added D7: Fan3100tsx, Package_TO_SOT_SMD:SOT-23-5, B.Cu at (214.9, 96.7)
- C11, D4: moved to B.Cu
- D5, D6: footprint LED_SMD:LED_0603_1608Metric -> LED_THT:LED_D3.0mm_Clear
- Q1, Q2: footprint Package_TO_SOT_THT:TO-220-3_Horizontal_TabDown -> Package_TO_SOT_THT:TO-247-3_Horizontal_TabDown
- R8: footprint Resistor_SMD:R_1206_3216Metric -> Resistor_SMD:R_0603_1608Metric
- moved R5 40.8 mm to (165.5, 123.9), turned to 270 degrees
- moved Q1 33.0 mm to (193.5, 92.4), turned to 0 degrees
- moved J3 32.4 mm to (124.0, 78.4), turned to 0 degrees
- moved R12 23.1 mm to (161.5, 129.5)
- moved R11 23.0 mm to (111.5, 121.5)
- moved J22 21.9 mm to (158.0, 118.0)
- moved U2 13.8 mm to (138.0, 108.8)
- moved J2 13.5 mm to (153.7, 130.2), turned to 270 degrees
- moved D3 12.9 mm to (214.0, 111.8), turned to 180 degrees
- moved J7 12.5 mm to (154.5, 81.5), turned to 315 degrees
- moved J12 12.2 mm to (181.7, 108.2), turned to 0 degrees
- moved Q3 10.2 mm to (219.0, 111.8)
- moved C8 10.0 mm to (218.5, 88.7), turned to 270 degrees
- moved J1 9.95 mm to (196.8, 107.0)
- moved R9 8.90 mm to (215.0, 87.9), turned to 270 degrees
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Routing:
- net Net-(J1-Pad1): track 72.8 -> 181.9 mm
- net Net-(J2-Pad1): track 115.1 -> 27.4 mm, vias 2 -> 0
- net GND: track 437.4 -> 362.0 mm
- net Net-(J3-Pad3): track 30.1 -> 97.7 mm, vias 0 -> 1
- net Net-(J3-Pad2): track 28.7 -> 89.9 mm, vias 0 -> 1
- net +3V3: track 248.5 -> 302.9 mm, vias 5 -> 4
- net MOSI: track 51.4 -> 104.5 mm, vias 2 -> 4
- net Net-(U2-Pad26): track 28.2 -> 58.4 mm
- net Net-(D6-Pad2): track 30.9 -> 3.91 mm, vias 1 -> 0
- net Net-(J7-Pad1): track 32.7 -> 59.4 mm, vias 0 -> 3
- net Net-(D7-Pad5): track 27.9 -> 52.5 mm, vias 1 -> 0
- net BLUE: track 18.9 -> 43.4 mm, vias 0 -> 2
- net Net-(D1-Pad2): track 31.5 -> 55.1 mm, vias 4 -> 2
- net Net-(U2-Pad8): track 24.6 -> 47.8 mm
- net RED: track 11.4 -> 29.9 mm
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Other:
- board size 132.8 x 68 mm -> 129 x 68 mm

Commit message: Add files via upload
Parts:
- C2, D1, D2, R11, R12, R6, R8: moved to B.Cu
- moved Q1 44.8 mm to (207.4, 135.0), turned to 180 degrees
- moved R9 42.6 mm to (177.5, 108.2)
- moved C8 40.1 mm to (180.5, 101.5)
- moved J11 36.8 mm to (213.3, 87.0), turned to 180 degrees
- moved J9 36.8 mm to (201.6, 87.0), turned to 180 degrees
- moved R4 36.7 mm to (200.5, 95.2), turned to 270 degrees
- moved J7 35.0 mm to (165.5, 114.8), turned to 270 degrees
- moved TH1 34.8 mm to (180.5, 107.5), turned to 90 degrees
- moved R6 33.9 mm to (203.5, 95.0), turned to 90 degrees
- moved D2 33.7 mm to (207.5, 97.0), turned to 270 degrees
- moved J3 32.9 mm to (152.5, 94.8), turned to 90 degrees
- moved C11 32.6 mm to (193.0, 104.0), turned to 270 degrees
- moved U3 32.0 mm to (190.5, 98.1), turned to 0 degrees
- moved D1 29.2 mm to (223.5, 94.6), turned to 0 degrees
- moved R8 26.6 mm to (211.3, 98.0), turned to 0 degrees
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Routing:
- net Net-(C1-Pad2): track 28.0 -> 195.4 mm, vias 0 -> 3
- net +3V3: track 302.9 -> 172.6 mm, vias 4 -> 2
- net Net-(J3-Pad3): track 97.7 -> 17.5 mm, vias 1 -> 0
- net Net-(J3-Pad2): track 89.9 -> 12.9 mm, vias 1 -> 0
- net Net-(U2-Pad12): track 101.4 -> 31.7 mm, vias 3 -> 1
- net GND: track 362.0 -> 424.8 mm
- net Net-(U2-Pad26): track 58.4 -> 7.26 mm
- net MOSI: track 104.5 -> 53.6 mm, vias 4 -> 0
- net Net-(R13-Pad2): track 25.8 -> 75.3 mm
- net Net-(J12-Pad3): track 52.1 -> 12.8 mm
- net Net-(D5-Pad2): track 41.7 -> 4.49 mm
- net Net-(U2-Pad8): track 47.8 -> 13.8 mm
- net Net-(D1-Pad3): track 4.26 -> 38.0 mm, vias 1 -> 2
- net cntrl: track 53.2 -> 22.6 mm
- net Net-(D7-Pad5): track 52.5 -> 81.4 mm
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Other:
- board size 129 x 68 mm -> 132.7 x 68 mm

Commit message: Add files via upload
Parts:
- removed J1: 220to12, Touch_pad:oblast_bp
- removed J11: 220v_OUT, Touch_pad:220V_1x02_P5.08mm_Horizontal
- removed J17, J18, J19: Conn_01x01, Touch_pad:polz_razjem
- removed J2: Prog, Connector_PinHeader_2.54mm:PinHeader_1x02_P2.54mm_Vertical_SMD_Pin1Left
- removed J22: SPI, Connector_PinHeader_2.54mm:PinHeader_1x04_P2.54mm_Vertical_SMD_Pin1Right
- removed J7: I2C, Connector_PinHeader_2.54mm:PinHeader_1x03_P2.54mm_Horizontal
- removed J9: 220v_IN, Touch_pad:220V_1x02_P5.08mm_Horizontal
- removed k1: Key, Touch_pad:TestPoint_Pad_1.0x1.0sm
- added I2C: I2C, Connector_PinHeader_2.54mm:PinHeader_1x03_P2.54mm_Horizontal, B.Cu at (84.7, 115.2)
- added IN: 220v_IN, SMout:OUT_IN(1), F.Cu at (201.9, 78.9)
- added Mode: Mode, SMout:2pins, F.Cu at (89.1, 133.5)
- added OUT: 220v_OUT, SMout:OUT_IN(1), F.Cu at (222.5, 78.9)
- added PS: 220to12, SMout:oblast_bp, F.Cu at (188.2, 95.1)
- added Prog: , SMout:2pins, F.Cu at (89.8, 133.4)
- added RST: Reset, SMout:polz_razjem, F.Cu at (84.0, 133.4)
- added SPI: SPI, Connector_PinHeader_2.54mm:PinHeader_1x04_P2.54mm_Vertical, B.Cu at (133.1, 133.9)
- C1, C2, C8: footprint Capacitor_SMD:C_1210_3225Metric -> Capacitor_SMD:C_0805_2012Metric
- C11: footprint Capacitor_SMD:C_1210_3225Metric -> Capacitor_SMD:C_0805_2012Metric; moved to F.Cu
- C4, R1, R5, TH2, U2: moved to B.Cu
- D5, D6: footprint LED_THT:LED_D3.0mm_Clear -> LED_SMD:LED_0805_2012Metric; moved to F.Cu
- J10: value Detect_nullA -> Pin; footprint Connector:FanPinHeader_1x03_P2.54mm_Vertical -> SMout:polz_razjem; moved to F.Cu
- J12: value Load_cntrlA -> Pin; footprint Connector:FanPinHeader_1x03_P2.54mm_Vertical -> SMout:polz_razjem; moved to F.Cu
- J13, J8: footprint Touch_pad:polz_razjem -> SMout:polz_razjem; moved to B.Cu
- J14: value Conn_01x01 -> Pin; footprint Touch_pad:polz_razjem -> SMout:polz_razjem; moved to B.Cu
- J15: value Conn_01x01 -> Pin; footprint Touch_pad:polz_razjem -> SMout:polz_razjem
- J16: value Conn_01x01 -> Conn_01x05; footprint Touch_pad:polz_razjem -> Connector_PinHeader_2.54mm:PinHeader_1x05_P2.54mm_Vertical; moved to B.Cu
- J4: value Mode -> Conn_01x05; footprint Connector_PinHeader_2.54mm:PinHeader_1x02_P2.54mm_Vertical_SMD_Pin1Left -> Connector_PinHeader_2.54mm:PinHeader_1x05_P2.54mm_Vertical
- J5: value Load_cntrl -> Pin; footprint Connector:FanPinHeader_1x03_P2.54mm_Vertical -> SMout:polz_razjem
- J6: value Detect_null -> Pin; footprint Connector:FanPinHeader_1x03_P2.54mm_Vertical -> SMout:polz_razjem
- R10: footprint Resistor_SMD:R_0603_1608Metric -> Resistor_SMD:R_1206_3216Metric
- R11, R12, k2, k3, k4, k5, k6, k7: moved to F.Cu
- R13, R2: footprint Resistor_SMD:R_0603_1608Metric -> Resistor_SMD:R_0805_2012Metric; moved to B.Cu
- R3: footprint OptoDevice:R_LDR_5.1x4.3mm_P3.4mm_Vertical -> SMout:R_LDR_5.1x4.3mm_P3.4mm_Vertical; moved to F.Cu
- R7: footprint Resistor_SMD:R_0603_1608Metric -> Resistor_SMD:R_2512_6332Metric
- R9: footprint Resistor_SMD:R_0603_1608Metric -> Resistor_SMD:R_0805_2012Metric
- RX0: renamed from J3; footprint Connector_PinHeader_2.54mm:PinHeader_1x04_P2.54mm_Horizontal -> Connector_PinHeader_2.54mm:PinHeader_1x04_P2.54mm_Vertical; moved to B.Cu
- SW_MODE: renamed from SW2; moved to F.Cu
- SW_RST: renamed from SW1; moved to F.Cu
- moved RX0 77.7 mm to (86.7, 136.0), turned to 270 degrees
- moved J10 74.8 mm to (145.6, 116.3)
- moved D6 69.9 mm to (132.7, 72.8), turned to 0 degrees
- moved J4 65.7 mm to (212.7, 129.5)
- moved SW_MODE 62.6 mm to (101.0, 135.3)
- moved R12 62.2 mm to (138.4, 72.8), turned to 180 degrees
- moved D5 60.5 mm to (100.2, 72.7), turned to 0 degrees
- moved TH2 55.2 mm to (102.3, 77.7), turned to 45 degrees
- moved R11 54.9 mm to (105.9, 72.7), turned to 180 degrees
- moved R13 50.6 mm to (105.0, 81.3), turned to 225 degrees
- moved Q1 46.6 mm to (189.3, 92.0), turned to 0 degrees
- moved J12 44.2 mm to (145.6, 118.8), turned to 0 degrees
- moved Q2 42.9 mm to (221.8, 92.0), turned to 180 degrees
- moved C8 37.6 mm to (211.8, 122.3), turned to 180 degrees
- moved TH1 35.1 mm to (210.8, 125.2), turned to 0 degrees
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Connections:
- net GPIO35 renamed photo
- D7 pad 3: cntrl -> Load_cntrl
- J12 pad 1: +3V3 -> Net-(J12-Pad1)
- J16 pad 1: Net-(J16-Pad1) -> +3V3
- J4 pad 1: Mode -> +3V3
- J4 pad 2: Net-(J4-Pad2) -> Load_cntrl
- J5 pad 1: +3V3 -> Net-(J5-Pad1)
- J6 pad 1: GPIO17 -> Net-(J6-Pad1)
- R9 pad 2: Net-(J12-Pad3) -> Net-(J4-Pad3)
- SW_MODE pad 2: Net-(J4-Pad2) -> Net-(J23-Pad2)
- TH1 pad 1: Net-(J12-Pad3) -> Net-(J4-Pad3)
- U2 pad 10: GPIO32 -> termo_bp
- U2 pad 11: GPIO26 -> cntrl
- U2 pad 17: Net-(J16-Pad1) -> Net-(J6-Pad1)
- U2 pad 18: Net-(J17-Pad1) -> Net-(J10-Pad1)
- U2 pad 19: Net-(J19-Pad1) -> Net-(J15-Pad1)
- U2 pad 20: Net-(J18-Pad1) -> Net-(J12-Pad1)
- U2 pad 22: Net-(J15-Pad1) -> Net-(J5-Pad1)
- U2 pad 28: GPIO17 -> null
- U4 pad 6: Net-(J10-Pad1) -> Detect_null
Routing:
- net GND: track 424.8 -> 161.7 mm, vias 4 -> 3
- net Net-(C1-Pad2): track 195.4 -> 20.7 mm, vias 3 -> 0
- net Net-(J1-Pad1): track 188.5 -> 39.7 mm, vias 1 -> 0
- net termo_bp: track 0.00 -> 122.1 mm, vias 0 -> 1
- net +3V3: track 172.6 -> 258.1 mm, vias 2 -> 5
- net null: track 0.00 -> 70.9 mm, vias 0 -> 1
- net cntrl: track 22.6 -> 90.8 mm
- net Net-(J16-Pad1): track 58.4 -> 0.00 mm
- net Net-(J19-Pad1): track 56.8 -> 0.00 mm
- net Net-(R13-Pad2): track 75.3 -> 18.9 mm
- net Net-(J17-Pad1): track 53.0 -> 0.00 mm
- net RED: track 48.7 -> 101.4 mm
- net Net-(J18-Pad1): track 45.8 -> 0.00 mm
- net Net-(U2-Pad8): track 13.8 -> 51.6 mm
- net Net-(C2-Pad2): track 70.7 -> 35.9 mm, vias 0 -> 2
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Other:
- board size 132.7 x 68 mm -> 156.1 x 68 mm
- board text added: "+12"
- board text added: "+3.3"
- board text added: "CLK"
- board text added: "CS"
- board text added: "Cntrl"
- board text added: "GND"
- board text added: "L"
- board text added: "MISO"
- board text added: "MOSI"
- board text added: "N"
- board text added: "Null"
- board text added: "SCL"
- board text added: "SDA"
- board text added: "Sw_M"
- board text added: "TX0"
- board text added: "Termo_PS"

Commit message: Add files via upload
Parts:
- removed TH1, TH2: Thermistor_NTC, Resistor_SMD:R_1206_3216Metric_Pad1.30x1.75mm_HandSolder
- added J17: I2C, Connector_PinHeader_2.54mm:PinHeader_1x03_P2.54mm_Vertical, F.Cu at (193.5, 125.5)
- added U1: LM75B, SMout:Diodes_SO-8, F.Cu at (210.5, 124.1)
- C11: moved to B.Cu
- J20: renamed from RST; value Reset -> Rst
- R13: footprint Resistor_SMD:R_0805_2012Metric -> Resistor_SMD:R_0603_1608Metric; moved to F.Cu
- R9: footprint Resistor_SMD:R_0805_2012Metric -> Resistor_SMD:R_0603_1608Metric
- moved R13 108.4 mm to (203.8, 126.0), turned to 180 degrees
- moved C8 6.75 mm to (218.5, 122.5), turned to 270 degrees
- moved R9 5.95 mm to (209.8, 119.5), turned to 180 degrees
- moved C11 0.66 mm to (202.5, 124.5)
- renumbered PS to J1, OUT to J11, SPI to J22, Mode to J23, RX0 to J3, I2C to J7, IN to J9, SW_RST to SW1, SW_MODE to SW2
Connections:
- J16 pad 3: termo_bp -> O.S.
- R13 pad 2: Net-(R13-Pad2) -> SCL
- R9 pad 2: Net-(J4-Pad3) -> SDA
- U2 pad 10: termo_bp -> Net-(U2-Pad10)
- U2 pad 26: Net-(U2-Pad26) -> O.S.
- U2 pad 6: Net-(R13-Pad2) -> Net-(U2-Pad6)
Routing:
- net termo_bp: track 122.1 -> 0.00 mm, vias 1 -> 0
- net O.S.: track 0.00 -> 77.4 mm, vias 0 -> 1
- net Net-(U2-Pad10): track 0.00 -> 54.2 mm
- net SDA: track 0.00 -> 19.0 mm
- net Net-(R13-Pad2): track 18.9 -> 0.00 mm
- net SCL: track 0.00 -> 17.2 mm
- net +3V3: track 258.1 -> 267.3 mm
- net GND: track 161.7 -> 160.0 mm
- net RED: track 101.4 -> 103.0 mm
- net Net-(U2-Pad24): track 42.2 -> 42.8 mm
- net +12V: track 38.0 -> 37.5 mm
- net Net-(J4-Pad3): track 7.39 -> 7.11 mm, vias 0 -> 1
Other:
- board text added: "O.S."

Commit message: Add files via upload
Parts:
- removed Prog: , SMout:2pins
- added J2: Prog, SMout:2pins, F.Cu at (89.6, 133.4)
- J17: footprint Connector_PinHeader_2.54mm:PinHeader_1x03_P2.54mm_Vertical -> Connector_PinSocket_2.54mm:PinSocket_1x03_P2.54mm_Vertical
- J3: footprint Connector_PinHeader_2.54mm:PinHeader_1x04_P2.54mm_Vertical -> SMout:4pins
Connections:
- U2 pad 10: Net-(U2-Pad10) -> (no net)
- U2 pad 32: Net-(U2-Pad32) -> (no net)
- U2 pad 6: Net-(U2-Pad6) -> (no net)
- U3 pad 4: Net-(U3-Pad4) -> (no net)
- U3 pad 5: Net-(U3-Pad5) -> (no net)
Routing:
- net Net-(U2-Pad10): track 54.2 -> 47.0 mm

Commit message: Add files via upload
Parts:
- moved J3 0.55 mm to (86.1, 136.0)
Routing:
- net Net-(J3-Pad3): track 36.6 -> 40.3 mm
- net +3V3: track 267.3 -> 270.5 mm
- net Net-(J3-Pad2): track 37.0 -> 38.9 mm
- net GND: track 160.0 -> 161.3 mm

Commit message: New regulator, buttons
Parts:
- removed J17: I2C, Connector_PinSocket_2.54mm:PinSocket_1x03_P2.54mm_Vertical
- removed J23: Mode, SMout:2pins
- removed J7: I2C, Connector_PinHeader_2.54mm:PinHeader_1x03_P2.54mm_Horizontal
- removed U3: L78L33_SO8, Package_SO:SOIC-8_3.9x4.9mm_P1.27mm
- added U22: AMS1117-3.3, Package_TO_SOT_SMD:SOT-223-3_TabPin2, B.Cu at (212.4, 119.8)
- C11: value 0.33mk -> 1uF
- C8: value 0.1mk -> 0.1uF
- J16, J4: value Conn_01x05 -> Conn_01x06; footprint Connector_PinHeader_2.54mm:PinHeader_1x05_P2.54mm_Vertical -> Connector_PinHeader_2.54mm:PinHeader_1x06_P2.54mm_Vertical
- Mode1: renamed from SW2; footprint Button_Switch_SMD:SW_DIP_SPSTx01_Slide_6.7x4.1mm_W6.73mm_P2.54mm_LowProfile_JPin -> Touch_pad:aLIEXPRESS_BUTTON_G71Y
- RST2: renamed from SW1; footprint Button_Switch_SMD:SW_DIP_SPSTx01_Slide_6.7x4.1mm_W6.73mm_P2.54mm_LowProfile_JPin -> Touch_pad:aLIEXPRESS_BUTTON_G71Y
- moved k3 18.5 mm to (103.5, 95.2), turned to 0 degrees
- moved J11 4.42 mm to (218.2, 80.0)
- moved RST2 2.88 mm to (83.8, 130.2), turned to 90 degrees
- moved C8 2.66 mm to (215.9, 122.1)
- moved C11 2.45 mm to (200.1, 124.7)
- moved J9 1.56 mm to (203.0, 80.0)
- moved Mode1 1.32 mm to (101.0, 134.0)
- moved R13 1.05 mm to (204.5, 126.8)
- renumbered J12 to CLK1, J15 to CMD1, J20 to RST1, J14 to SD0, J5 to SD1, J6 to SD2, J10 to SD3, J13 to S_VN1, J8 to S_VP1
Connections:
- J16 pad 3: O.S. -> null
- J16 pad 4: null -> SCL
- J16 pad 5: GND -> SDA
- J4 pad 3: Net-(J4-Pad3) -> Detect_null
- J4 pad 4: Detect_null -> SCL
- J4 pad 5: GND -> SDA
- Mode1 pad 2: Net-(J23-Pad2) -> Mode
- R2 pad 2: Net-(J20-Pad1) -> Net-(R2-Pad2)
- RST1 pad 1: Net-(J20-Pad1) -> Net-(R2-Pad2)
- RST2 pad 1: GND -> Net-(R2-Pad2)
- RST2 pad 2: Net-(J20-Pad1) -> GND
- U1 pad 3: Net-(J4-Pad3) -> (no net)
- U2 pad 26: O.S. -> (no net)
- U2 pad 3: Net-(J20-Pad1) -> Net-(R2-Pad2)
- U2 pad 33: Net-(J7-Pad1) -> SDA
- U2 pad 36: Net-(J7-Pad2) -> SCL
Routing:
- net Net-(R2-Pad2): track 0.00 -> 78.4 mm, vias 0 -> 1
- net O.S.: track 77.4 -> 0.00 mm, vias 1 -> 0
- net Net-(J20-Pad1): track 75.1 -> 0.00 mm, vias 1 -> 0
- net Net-(U2-Pad10): track 47.0 -> 0.00 mm
- net SDA: track 19.0 -> 51.0 mm
- net Net-(J7-Pad1): track 30.5 -> 0.00 mm
- net Net-(J7-Pad2): track 26.6 -> 0.00 mm
- net SCL: track 17.2 -> 38.8 mm, vias 0 -> 2
- net Mode: track 63.5 -> 78.1 mm, vias 0 -> 1
- net Net-(D7-Pad5): track 59.7 -> 73.8 mm
- net Net-(J3-Pad3): track 40.3 -> 50.5 mm, vias 0 -> 1
- net Net-(J3-Pad2): track 38.9 -> 48.7 mm
- net +3V3: track 270.5 -> 261.0 mm, vias 5 -> 8
- net Net-(J23-Pad2): track 9.26 -> 0.00 mm
- net MOSI: track 59.3 -> 50.4 mm
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Other:
- board text added: "CTRL"
- board text added: "NULL"
- board text added: "PROG"
- board text added: "RX0"
- board text removed: "Null"
- board text removed: "O.S."
- board text removed: "Sw_M"
- board text removed: "Termo_PS"
